Commit message: Basic CMakeLists for generating robots files for the package

File: scara/scara.urdf (robot description, URDF)
Before this commit: robot None, 0 links, 0 joints
Links:
- added link base, mass 0.0; collision box size=0.0 0.0 0.0; visual mesh filename=package://simple_robots/scara/meshs/base.dae scale=1.0

Commit message: Basic SCARA - Basic simulator (that doesn't accept any input yet) - Launch file for the SCARA environment

File: scara/scara.urdf (robot description, URDF)
Before this commit: robot sr-scara, 1 links, 0 joints
Links:
- removed link base
- added link base_link; collision box size=0.0 0.0 0.0; visual mesh filename=package://simple_robots/scara/meshs/base.dae scale=1.0 1.0 1.0
- added link link1, mass 1.0; visual mesh filename=package://simple_robots/scara/meshs/link1.dae scale=1.0 1.0 1.0
- added link link2, mass 1.0; visual mesh filename=package://simple_robots/scara/meshs/link2.dae scale=1.0 1.0 1.0
- added link link3
- added link link4, mass 1.0; visual mesh filename=package://simple_robots/scara/meshs/link3.dae scale=1.0 1.0 1.0
Joints:
- added joint joint1: type revolute, parent base_link, child link1, origin xyz=0.0 0.0 0.18 rpy=0.0 0.0 0.0, axis 0.0 0.0 1.0, limit lower=-3.14 upper=3.140 effort=0.0 velocity=0.0
- added joint joint2: type revolute, parent link1, child link2, origin xyz=0.15 0.0 0.0 rpy=0.0 0.0 0.0, axis 0.0 0.0 1.0, limit lower=-1.57 upper=1.57 effort=0.0 velocity=0.0
- added joint joint3: type revolute, parent link2, child link3, origin xyz=0.10 0.0 0.0 rpy=0.0 0.0 0.0, axis 0.0 0.0 1.0, limit lower=-3.14 upper=3.140 effort=0.0 velocity=0.0
- added joint joint4: type prismatic, parent link3, child link4, origin xyz=0.0 0.0 0.0 rpy=3.14 0.0 0.0, axis 0.0 0.0 1.0, limit lower=0 upper=0.096 effort=0.0 velocity=0.0

Commit message: Scaled up SCARA version

File: scara/scara.urdf (robot description, URDF)
Before this commit: robot sr-scara, 5 links, 4 joints
Joints:
- joint joint1: origin xyz=0.0 0.0 0.18 rpy=0.0 0.0 0.0 -> xyz=0.0 0.0 0.94 rpy=0.0 0.0 0.0
- joint joint2: origin xyz=0.15 0.0 0.0 rpy=0.0 0.0 0.0 -> xyz=0.5 0.0 0.0 rpy=0.0 0.0 0.0
- joint joint3: origin xyz=0.10 0.0 0.0 rpy=0.0 0.0 0.0 -> xyz=0.5 0.0 0.0 rpy=0.0 0.0 0.0
- joint joint4: limit lower=0 upper=0.096 effort=0.0 velocity=0.0 -> lower=0 upper=0.716 effort=0.0 velocity=0.0
